File: pmt-plugin-board.kicad_pcb (KiCad board)
At the start: 2 copper layers, 29 x 35 mm, 21 parts, among them J1 CONN_ARDUINO, J2 CONN_ISP, J3 PMT Connector, J4 12V In, U1 5V Regulator, U2 ATMEGA328P-AU, Y1 Resonator

Commit message: Add gerber files
Parts:
- moved JP1 1.34 mm to (150.5, 97.8), turned to 90 degrees
Changed lines of the file:
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@@
   (general
     (links 52)
-    (no_connects 0)
-    (area 132.924999 70.924999 166.075001 106.075001)
+    (no_connects 1)
+    (area 132.875 70.899999 162.075001 106.075001)
     (thickness 1.6)
     (drawings 5)
@@
       (psa4output false)
       (plotreference true)
-      (plotvalue true)
+      (plotvalue false)
       (plotinvisibletext false)
       (padsonsilk false)
@@
       (outputformat 1)
       (mirror false)
-      (drillshape 1)
+      (drillshape 0)
       (scaleselection 1)
-      (outputdirectory ""))
+      (outputdirectory gerber/))
   )
   (net 0 "")
@@
   )
   (module Resistors_SMD:R_0805 (layer F.Cu)
-    (at 149.55 98.8 180)
+    (at 150.5 97.85 90)
     (descr "Resistor SMD 0805, reflow soldering, Vishay (see dcrcw.pdf)")
     (tags "resistor 0805")
     (attr smd)
-    (fp_text reference JP1 (at 0 1.5 180) (layer F.SilkS)
-      (effects (font (size 1 1) (thickness 0.15)))
-    )
-    (fp_text value 3.3V-3.3V_USB (at -1.25 -1.6 180) (layer F.Fab)
+    (fp_text reference JP1 (at 0 1.5 90) (layer F.SilkS)
+      (effects (font (size 1 1) (thickness 0.15)))
+    )
+    (fp_text value 3.3V-3.3V_USB (at -1.25 -1.6 90) (layer F.Fab)
       (effects (font (size 1 1) (thickness 0.15)))
     )
@@
     (fp_line (start 1.55 0.9) (end 1.55 -0.9) (layer F.CrtYd) (width 0.05))
     (fp_line (start 1.55 0.9) (end -1.55 0.9) (layer F.CrtYd) (width 0.05))
-    (pad 1 smd rect (at -0.95 0 180) (size 0.7 1.3) (layers F.Cu F.Paste F.Mask)
+    (pad 1 smd rect (at -0.95 0 90) (size 0.7 1.3) (layers F.Cu F.Paste F.Mask)
       (net 9 +3.3V_USB))
-    (pad 2 smd rect (at 0.95 0 180) (size 0.7 1.3) (layers F.Cu F.Paste F.Mask)
+    (pad 2 smd rect (at 0.95 0 90) (size 0.7 1.3) (layers F.Cu F.Paste F.Mask)
       (net 1 +3.3V))
     (model ${KISYS3DMOD}/Resistors_SMD.3dshapes/R_0805.wrl
